File: schematic/polypoop/control-switches.kicad_sch (KiCad schematic)
At the start: 12 parts, among them SW1 SW_Push_DPDT, SW2 SW_Push, SW3 SW_Push_DPDT, SW4 SW_Push, SW5 SW_Push_DPDT, SW6 SW_Push, SW7 SW_Push_DPDT, SW8 SW_Push

Commit message: update
Other:
- note added: "Управляющий сигнал подтягивается через резистор к одному состоянию (вкл или выкл) и кнопкой переключается на другое (выкл или вкл). Тумблер меняет состояния местами. Таким образом, переключение тумблера в противоположное состояние как и нажатие/отжатие кнопки переключают свою цепочку осцилляторов в противоположное текущему состояние."
- title: (none) -> Переключатели управления цепочками осцилляторов
Changed lines of the file:
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@@
 	(generator_version "10.0")
 	(paper "A4")
+	(title_block
+		(title "Переключатели управления цепочками осцилляторов")
+	)
+	(text "Управляющий сигнал подтягивается через резистор к одному состоянию\n(вкл или выкл) и кнопкой переключается на другое (выкл или вкл).\n\nТумблер меняет состояния местами.\n\nТаким образом, переключение тумблера в противоположное состояние\nкак и нажатие/отжатие кнопки переключают свою цепочку осцилляторов\nв противоположное текущему состояние."
+		(exclude_from_sim no)
+		(at 90.424 41.91 0)
+		(effects
+			(font
+				(size 1.27 1.27)
+			)
+			(justify left)
+		)
+	)
 	(junction
 		(at 107.95 125.73)
