File: schematic/polypoop/osc-1-2.kicad_sch (KiCad schematic)
At the start: 32 parts, among them U1 NE556, U2 NE556, U3 NE556, U7 4066

Commit message: update
Parts:
- removed C3, C6: 39nF, symbol Device:C_Polarized
- added C21, C22: 39nF, symbol Device:C
- added D1, D2, D3, D4: LED, symbol Device:LED
- added R40, R50, R51, R52: 10K, symbol Device:R_US
- U7: value 4066 -> К561КТ3А
Connections:
- net +12V: now also R40.1, R50.1, R51.1, R52.1
- net GND: now also C21.1, C22.1
- net at R6.1, U3.2 (THRES), U3.6 (TRIG): now also C21.2
- net at R12.1, U3.12 (THRES), U3.8 (TRIG): now also C22.2
- net at U2.13 (DISCH): now also D2.1 (K)
- net at U2.1 (DISCH): now also D1.1 (K)
- net at U1.1 (DISCH): now also D3.1 (K)
- net at U1.13 (DISCH): now also D4.1 (K)
- new net: D3.2 (A), R51.2
- new net: D1.2 (A), R40.2
- new net: D4.2 (A), R52.2
- new net: D2.2 (A), R50.2
- no-connect marks 0 -> 2
Other:
- note added: "Аналоговые переключатели U7(A..D) подключают выходы каждого осциллятора к входу выходного усилителя только когда осциллятор активен. Таким образом, неактивные осцилляторы не подтягивают выход в одну сторону, сигнал всегда колеблется симметрично относительно среднего уровня (V_{Ref} ~= 6V). Согласно документации, К561КТ3 должна подтягивать вход к земле когда переключатель выключен. На практике это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"
- title: (none) -> Осцилляторы 1 и 2
