File: schematic/polypoop/osc-3-4.kicad_sch (KiCad schematic)
At the start: 32 parts, among them U4 NE556, U5 NE556, U6 NE556, U7 4066

Commit message: update
Parts:
- removed C11, C12: 39nF, symbol Device:C_Polarized
- added C23, C24: 39nF, symbol Device:C
- added D5, D6, D7, D8: LED, symbol Device:LED
- added R53, R54, R55, R56: 10K, symbol Device:R_US
- U7: value 4066 -> К561КТ3А
Connections:
- net +12V: now also R53.1, R54.1, R55.1, R56.1
- net GND: now also C23.1, C24.1
- net at U4.1 (DISCH): now also D5.1 (K)
- net at R24.1, U6.2 (THRES), U6.6 (TRIG): now also C23.2
- net at U4.13 (DISCH): now also D6.1 (K)
- net at U5.1 (DISCH): now also D7.1 (K)
- net at U5.13 (DISCH): now also D8.1 (K)
- net at R26.1, U6.12 (THRES), U6.8 (TRIG): now also C24.2
- new net: D6.2 (A), R54.2
- new net: D8.2 (A), R56.2
- new net: D5.2 (A), R53.2
- new net: D7.2 (A), R55.2
Other:
- title: (none) -> Осцилляторы 3 и 4
