File: schematic/polypoop/output-amplifier.kicad_sch (KiCad schematic)
At the start: 12 parts, among them J1 AudioJack2_Ground_Switch, U8 TL074

Commit message: update
Parts:
- removed R40: 10K, symbol Device:R_US
- added C19: 100nF, symbol Device:C
- added C20: 220nF, symbol Device:C
- added R48: 4K7, symbol Device:R_US
- added R49: 100R, symbol Device:R_US
- R41: value 10K -> 1k
- R47: value 10K -> 4K7
- RV13: value R_Potentiometer_US -> 4K7
Connections:
- net GND: no longer RV13.3
- net IN: now also R41.2, U8.2 (-)
- net V_Ref: now also RV13.3
- net at C13.2, R39.2: now also C20.1
- net at J1.T, R38.2, R39.1: now also C20.2
- net at R42.2, R47.1, U8.6 (-): now also C19.2, R48.1
- net at R47.2, RV13.2: now also C19.1, R48.2
- net at R41.1, U8.1: now also R49.2; no longer RV13.1
- new net: R49.1, RV13.1
Other:
- note added: "Конденсаторы C19 и C20 увеличивают содержание высоких частот в сигнале - усилитель работает как ФВЧ (high-pass filter). Это нужно чтобы получить большую громкость пъезоизлучателя."
- title: (none) -> Промежуточный и выходной усилители
- moved on the sheet: R42, R47, U8B
