File: schematic/polypoop/pitch-control.kicad_sch (KiCad schematic)
At the start: 5 parts, among them U8 TL074

Commit message: update
Connections:
- net +12V: now also RV16.1
- net GND: now also RV15.3
Other:
- note added: "Подстроечники RV15 и RV16 определяют верхний и нижний предел регулировки тона. В верхнее и нижнее положение можно поменять местами соответствующей настройкой этих подстроечников."
- title: (none) -> Регулятор тона
- moved on the sheet: RV15
Changed lines of the file:
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@@
 	(generator_version "10.0")
 	(paper "A4")
+	(title_block
+		(title "Регулятор тона")
+	)
+	(text "Подстроечники RV15 и RV16 определяют\nверхний и нижний предел регулировки тона.\n\nВ верхнее и нижнее положение можно поменять местами\nсоответствующей настройкой этих подстроечников."
+		(exclude_from_sim no)
+		(at 82.804 72.39 0)
+		(effects
+			(font
+				(size 1.27 1.27)
+			)
+			(justify left)
+		)
+	)
+	(junction
+		(at 101.6 120.65)
+		(diameter 0)
+		(color 0 0 0 0)
+	)
 	(junction
 		(at 146.05 101.6)
@@
 		(color 0 0 0 0)
 	)
+	(junction
+		(at 76.2 82.55)
+		(diameter 0)
+		(color 0 0 0 0)
+	)
 	(wire
 		(pts
@@
 	(wire
 		(pts
+			(xy 101.6 110.49) (xy 101.6 82.55)
+		)
+		(stroke
+			(width 0)
+			(type default)
+		)
+	)
+	(wire
+		(pts
 			(xy 130.81 101.6) (xy 146.05 101.6)
 		)
@@
 	(wire
 		(pts
-			(xy 101.6 92.71) (xy 101.6 110.49)
-		)
-		(stroke
-			(width 0)
-			(type default)
-		)
-	)
-	(wire
-		(pts
 			(xy 184.15 116.84) (xy 184.15 104.14)
 		)
@@
 	(wire
 		(pts
+			(xy 76.2 82.55) (xy 76.2 85.09)
+		)
+		(stroke
+			(width 0)
+			(type default)
+		)
+	)
+	(wire
+		(pts
+			(xy 76.2 120.65) (xy 101.6 120.65)
+		)
+		(stroke
+			(width 0)
+			(type default)
+		)
+	)
+	(wire
+		(pts
 			(xy 179.07 104.14) (xy 184.15 104.14)
 		)
@@
 	(wire
 		(pts
-			(xy 101.6 76.2) (xy 101.6 85.09)
+			(xy 76.2 76.2) (xy 76.2 82.55)
 		)
 		(stroke
@@
 	(wire
 		(pts
+			(xy 101.6 82.55) (xy 76.2 82.55)
+		)
+		(stroke
+			(width 0)
+			(type default)
+		)
+	)
+	(wire
+		(pts
 			(xy 146.05 101.6) (xy 163.83 101.6)
 		)
@@
 	(wire
 		(pts
-			(xy 105.41 88.9) (xy 127 88.9)
+			(xy 80.01 88.9) (xy 127 88.9)
 		)
 		(stroke
@@
 	(wire
 		(pts
-			(xy 101.6 118.11) (xy 101.6 127)
+			(xy 101.6 120.65) (xy 101.6 127)
+		)
+		(stroke
+			(width 0)
+			(type default)
+		)
+	)
+	(wire
+		(pts
+			(xy 76.2 92.71) (xy 76.2 120.65)
+		)
+		(stroke
+			(width 0)
+			(type default)
+		)
+	)
+	(wire
+		(pts
+			(xy 101.6 118.11) (xy 101.6 120.65)
 		)
 		(stroke
@@
 	(symbol
 		(lib_id "power:+12V")
-		(at 101.6 76.2 0)
+		(at 76.2 76.2 0)
 		(unit 1)
 		(body_style 1)
@@
 		(fields_autoplaced yes)
 		(property "Reference" "#PWR062"
-			(at 101.6 80.01 0)
+			(at 76.2 80.01 0)
 			(hide yes)
 			(show_name no)
@@
 		)
 		(property "Value" "+12V"
-			(at 101.6 71.12 0)
+			(at 76.2 71.12 0)
 			(show_name no)
 			(do_not_autoplace no)
@@
 		)
 		(property "Footprint" ""
-			(at 101.6 76.2 0)
+			(at 76.2 76.2 0)
 			(hide yes)
 			(show_name no)
@@
 		)
 		(property "Datasheet" ""
-			(at 101.6 76.2 0)
+			(at 76.2 76.2 0)
 			(hide yes)
 			(show_name no)
@@
 		)
 		(property "Description" "Power symbol creates a global label with name \"+12V\""
-			(at 101.6 76.2 0)
+			(at 76.2 76.2 0)
 			(hide yes)
 			(show_name no)
@@
 	(symbol
 		(lib_id "Device:R_Potentiometer_Trim_US")
-		(at 101.6 88.9 0)
+		(at 76.2 88.9 0)
 		(unit 1)
 		(body_style 1)
@@
 		(fields_autoplaced yes)
 		(property "Reference" "RV15"
-			(at 99.06 87.6299 0)
+			(at 73.66 87.6299 0)
 			(show_name no)
 			(do_not_autoplace no)
@@
 		)
 		(property "Value" "10K"
-			(at 99.06 90.1699 0)
+			(at 73.66 90.1699 0)
 			(show_name no)
 			(do_not_autoplace no)
@@
 		)
 		(property "Footprint" ""
-			(at 101.6 88.9 0)
+			(at 76.2 88.9 0)
 			(hide yes)
 			(show_name no)
@@
 		)
 		(property "Datasheet" ""
-			(at 101.6 88.9 0)
+			(at 76.2 88.9 0)
 			(hide yes)
 			(show_name no)
@@
 		)
 		(property "Description" "Trim-potentiometer, US symbol"
-			(at 101.6 88.9 0)
+			(at 76.2 88.9 0)
 			(hide yes)
 			(show_name no)
@@
 		)
 		(property "Sim.Device" "R"
-			(at 101.6 88.9 0)
+			(at 76.2 88.9 0)
 			(hide yes)
 			(show_name no)
@@
 		)
 		(property "Sim.Type" "POT"
-			(at 101.6 88.9 0)
+			(at 76.2 88.9 0)
 			(hide yes)
 			(show_name no)
@@
 		)
 		(property "Sim.Pins" "1=r0 2=wiper 3=r1"
-			(at 101.6 88.9 0)
-			(hide yes)
-			(show_name no)
+			(at 76.2 88.9 0)
+			(hide yes)
+			(show_name no)
