File: schematic/polypoop/power.kicad_sch (KiCad schematic)
At the start: 12 parts, among them J2 USB_C_Receptacle, SW9 SW_SPST, U8 TL074, U9 L7812

Commit message: update
Other:
- note added: "V_{Ref} - псевдо-нулевая точка между землёй и напряжением питания - необходима для работы усилителей при однополярном питании."
- note added: "Напряжение в 5V с USB-порта сначала преобразуется в повышенное напряжение, около 15V, затем стабилизируется линейным стабилизатором до уровня 12V. Это позволяет устройству работать стабильно при колебаниях напряжения на входе. Линейный стабилизатор более жёстко фиксирует напряжение питания и подавляет часть высокочастотных пульсаций от импульсного преобразователя."
- note added: "Переключатель питания - часть регулятора громкости"
- title: (none) -> Цепи питания
Changed lines of the file:
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@@
 	(generator_version "10.0")
 	(paper "A4")
+	(title_block
+		(title "Цепи питания")
+	)
 	(rectangle
 		(start 114.3 44.45)
@@
 		(effects
 			(font
+				(size 1.27 1.27)
+			)
+		)
+	)
+	(text "Напряжение в 5V с USB-порта сначала преобразуется в\nповышенное напряжение, около 15V, затем стабилизируется\nлинейным стабилизатором до уровня 12V.\n\nЭто позволяет устройству работать стабильно\nпри колебаниях напряжения на входе.\nЛинейный стабилизатор более жёстко фиксирует напряжение\nпитания и подавляет часть высокочастотных пульсаций от\nимпульсного преобразователя."
+		(exclude_from_sim no)
+		(at 113.792 30.734 0)
+		(effects
+			(font
+				(size 1.27 1.27)
+			)
+			(justify left)
+		)
+	)
+	(text "V_{Ref} - псевдо-нулевая точка между землёй и\nнапряжением питания - необходима для работы\nусилителей при однополярном питании."
+		(exclude_from_sim no)
+		(at 175.514 141.224 0)
+		(effects
+			(font
+				(size 1.27 1.27)
+			)
+			(justify left)
+		)
+	)
+	(text "Переключатель питания\n-\nчасть регулятора громкости"
+		(exclude_from_sim no)
+		(at 93.218 58.42 0)
+		(effects
+			(font
